Commit message: Updated robot base and camera position in sim

File: ros2_ws/src/tidybot_description/urdf/tidybot_wx200.urdf.xacro (robot description, xacro)
@@ -14,5 +14,5 @@
     <visual>
       <geometry>
-        <mesh filename="${mesh_path}/base/new_tidybot.stl" scale="0.001 0.001 0.001"/>
+        <mesh filename="${mesh_path}/base/Crab_Base.stl" scale="0.001 0.001 0.001"/>
       </geometry>
       <material name="silver"/>
@@ -20,5 +20,5 @@
     <collision>
       <geometry>
-        <mesh filename="${mesh_path}/base/new_tidybot.stl" scale="0.001 0.001 0.001"/>
+        <mesh filename="${mesh_path}/base/Crab_Base.stl" scale="0.001 0.001 0.001"/>
       </geometry>
     </collision>
@@ -35,18 +35,22 @@
     <child link="base_link"/>
   </joint>
-  <!-- ==================== CAMERA TOWER (EXTRUSION) ==================== -->
-  <link name="camera_tower">
-    <visual>
-      <origin xyz="0.13 -0.01 0.3847" rpy="0 0 1.5708"/>
-      <geometry>
-        <mesh filename="${mesh_path}/base/2020_extrusion_250mm.stl" scale="0.001 0.001 0.001"/>
-      </geometry>
-      <material name="silver"/>
-    </visual>
-  </link>
-  <joint name="base_to_camera_tower" type="fixed">
+  <!-- ==================== CAMERA MOUNT ==================== -->
+  <link name="camera_mount">
+    <visual>
+      <geometry>
+        <mesh filename="${mesh_path}/base/Camera_Mount_v3.stl" scale="0.001 0.001 0.001"/>
+      </geometry>
+      <material name="dark_grey"/>
+    </visual>
+    <inertial>
+      <origin xyz="0 0 0"/>
+      <mass value="0.1"/>
+      <inertia ixx="0.0001" ixy="0" ixz="0" iyy="0.0001" iyz="0" izz="0.0001"/>
+    </inertial>
+  </link>
+  <joint name="base_to_camera_mount" type="fixed">
     <parent link="base_link"/>
-    <child link="camera_tower"/>
-    <origin xyz="0 0 0" rpy="0 0 0"/>
+    <child link="camera_mount"/>
+    <origin xyz="0 -0.1125 0.279" rpy="0 0 -1.5708"/>
   </joint>
   <!-- ==================== PAN-TILT CAMERA SYSTEM ==================== -->
@@ -66,7 +70,7 @@
   </link>
   <joint name="camera_pan" type="revolute">
-    <parent link="base_link"/>
+    <parent link="camera_mount"/>
     <child link="pan_link"/>
-    <origin xyz="0.12 0 0.6347" rpy="0 0 0"/>
+    <origin xyz="0 0 0" rpy="0 0 0"/>
     <axis xyz="0 0 1"/>
     <limit lower="-1.5708" upper="1.5708" effort="2" velocity="1.0"/>
@@ -127,5 +131,5 @@
   </joint>
   <!-- ==================== WX200 ARM MACRO ==================== -->
-  <xacro:macro name="wx200_arm" params="prefix y_offset">
+  <xacro:macro name="wx200_arm" params="prefix x_offset y_offset yaw">
     <link name="${prefix}_arm_base_link">
       <visual>
@@ -141,5 +145,5 @@
       <parent link="base_link"/>
       <child link="${prefix}_arm_base_link"/>
-      <origin xyz="0.1199 ${y_offset} 0.3847" rpy="0 0 0"/>
+      <origin xyz="${x_offset} ${y_offset} 0.3847" rpy="0 0 ${yaw}"/>
     </joint>
     <link name="${prefix}_shoulder_link">
@@ -339,5 +343,5 @@
   </xacro:macro>
   <!-- Instantiate both arms -->
-  <xacro:wx200_arm prefix="right" y_offset="-0.15"/>
-  <xacro:wx200_arm prefix="left" y_offset="0.15"/>
+  <xacro:wx200_arm prefix="right" x_offset="0.15" y_offset="-0.1199" yaw="-1.5708"/>
+  <xacro:wx200_arm prefix="left" x_offset="-0.15" y_offset="-0.1199" yaw="-1.5708"/>
 </robot>
