Commit message: Revert base_to_camera_mount yaw to -90deg; add camera_mount_urdf_issue.md
Commit 3cee5a4 changed the joint from rpy='0 0 -1.5708' to rpy='0 0 0', which
rotated the entire camera TF chain 90deg from physical reality. This caused all
3D object poses from detect_object_real.py to be wrong (x/y swapped/flipped),
breaking test_pickup.py grasp targets.

Reverted to rpy='0 0 -1.5708' which matches the physical mount orientation
(camera faces forward at pan=0). Added docs explaining the issue and the
separate tilt sign bug.

File: ros2_ws/src/tidybot_description/urdf/tidybot_wx250s.urdf.xacro (robot description, xacro)
@@ -55,5 +55,5 @@
     <parent link="base_link"/>
     <child link="camera_mount"/>
-    <origin xyz="0 -0.1125 0.279" rpy="0 0 0"/>
+    <origin xyz="0 -0.1125 0.279" rpy="0 0 -1.5708"/>  <!-- -90° yaw matches physical mount orientation -->
   </joint>
   <!-- ==================== TOP SENSOR STACK (SHARED EXTRUSION + LIDAR + TOP CAMERA) ==================== -->
